File: Ori.kicad_sch (KiCad schematic)
At the start: 93 parts, among them U3 LSM6DS3TR-C, Y1 26MHz, Y2 24MHz, Y3 32.768KHz

Commit message: test2
Parts:
- removed C22, C23, C25: 0.1uF, symbol Device:C_Small
- removed C30: 10uF, symbol Device:C_Small
- removed C33: 1uF, symbol Device:C_Small
- removed R6: 10k, symbol Device:R
- removed unit 3 of U1
- removed U10, U11, U8, U9: ~, Ori_components:PESD5V0S1BSF, symbol Ori_Components:PESD5V0S1BSF
- removed U2: ~, Ori_components:QFN-24-1EP_4x4mm_P0.5mm_EP2.8x2.8mm, symbol Ori_Components:ESP8684
- removed unit 3 of U3
- removed unit 2 of U3
- removed U4: ~, Ori_components:4 pin WLCPS, symbol Ori_Components:QMC6309
- removed unit 3 of U6
- removed unit 19 of U6
- removed unit 4 of U7
- removed unit 3 of U7
- added C19, C20: 1uF, Capacitor_SMD:C_0402_1005Metric, symbol Device:C_Small
- added C32, C35, C68, C69, C70, C71, C72: 100nF, Capacitor_SMD:C_0402_1005Metric, symbol Device:C_Small
- added C37: 820pF, Capacitor_SMD:C_0402_1005Metric, symbol Device:C_Small
- added C40, C42: 4.7uF, Capacitor_SMD:C_0402_1005Metric, symbol Device:C_Small
- added L7: 15nH, Capacitor_SMD:C_0402_1005Metric, symbol Device:L_Small
- added MIC1: ~, Ori_components:MMICT390200012, symbol Ori_Components:MMICT390200012
- added R1: 4.7k, Capacitor_SMD:C_0402_1005Metric, symbol Device:R
- added SW1: RotaryEncoder_Switch, symbol Device:RotaryEncoder_Switch
- added unit 5 of U2
- added U3: ~, Ori_components:nRF52840_wlcsp, symbol Ori_Components:nRF52840
- added U6: ~, Ori_components:4 pin WLCPS, symbol Ori_Components:AK09918C
- C1: renamed from C3; footprint (none) -> Capacitor_SMD:C_0402_1005Metric
- C10: renamed from C85; footprint (none) -> Capacitor_SMD:C_0402_1005Metric
- C11: renamed from C86; footprint (none) -> Capacitor_SMD:C_0402_1005Metric
- C12: renamed from C48; footprint (none) -> Capacitor_SMD:C_0402_1005Metric
- C13: renamed from C49; footprint (none) -> Capacitor_SMD:C_0402_1005Metric
- C14: renamed from C50; footprint (none) -> Capacitor_SMD:C_0402_1005Metric
- C15: renamed from C41; footprint (none) -> Capacitor_SMD:C_0402_1005Metric
- C16: renamed from C40; value 0.1uF -> 100nF; footprint (none) -> Capacitor_SMD:C_0402_1005Metric
- C17: renamed from C60; value 0.1uF -> 100nF; footprint (none) -> Capacitor_SMD:C_0402_1005Metric
- C18: renamed from C28; footprint (none) -> Capacitor_SMD:C_0402_1005Metric
- C2: renamed from C4; footprint (none) -> Capacitor_SMD:C_0402_1005Metric
- C21: renamed from C32; footprint (none) -> Capacitor_SMD:C_0402_1005Metric
- C22: renamed from C43; footprint (none) -> Capacitor_SMD:C_0402_1005Metric
- C23: renamed from C27; footprint (none) -> Capacitor_SMD:C_0402_1005Metric
- C24: value 0.1uF -> 47nF; footprint (none) -> Capacitor_SMD:C_0402_1005Metric
- C25: renamed from C51; footprint (none) -> Capacitor_SMD:C_0402_1005Metric
- C26: value 10uF -> 100nF; footprint (none) -> Capacitor_SMD:C_0402_1005Metric
- C27: renamed from C42; footprint (none) -> Capacitor_SMD:C_0402_1005Metric
- C28: renamed from C61; value 0.1uF -> 100nF; footprint (none) -> Capacitor_SMD:C_0402_1005Metric
- C29: value 2.2uF -> 4.7uF; footprint (none) -> Capacitor_SMD:C_0402_1005Metric
- C3: renamed from C2; footprint (none) -> Capacitor_SMD:C_0402_1005Metric
- C30: renamed from C52; footprint (none) -> Capacitor_SMD:C_0402_1005Metric
- C31: value 10nF -> 100nF; footprint (none) -> Capacitor_SMD:C_0402_1005Metric
- C33: renamed from C36; footprint (none) -> Capacitor_SMD:C_0402_1005Metric
- C34: renamed from C53; value 2.2uF -> 4.7uF; footprint (none) -> Capacitor_SMD:C_0402_1005Metric
- C36: renamed from C37; footprint (none) -> Capacitor_SMD:C_0402_1005Metric
- C38: renamed from C62; value 0.1uF -> 100nF; footprint (none) -> Capacitor_SMD:C_0402_1005Metric
- C39: renamed from C54; value 2.2uF -> 4.7uF; footprint (none) -> Capacitor_SMD:C_0402_1005Metric
- C4: renamed from C1; footprint (none) -> Capacitor_SMD:C_0402_1005Metric
- C41: renamed from C73; footprint (none) -> Capacitor_SMD:C_0402_1005Metric
- C43: renamed from C55; footprint (none) -> Capacitor_SMD:C_0402_1005Metric
- C44: renamed from C63; value 0.1uF -> 100nF; footprint (none) -> Capacitor_SMD:C_0402_1005Metric
- C45: renamed from C74; footprint (none) -> Capacitor_SMD:C_0402_1005Metric
- C46: renamed from C56; footprint (none) -> Capacitor_SMD:C_0402_1005Metric
- C47: renamed from C57; footprint (none) -> Capacitor_SMD:C_0402_1005Metric
- C48: renamed from C77; footprint (none) -> Capacitor_SMD:C_0402_1005Metric
- C49: renamed from C64; value 0.1uF -> 100nF; footprint (none) -> Capacitor_SMD:C_0402_1005Metric
- C5, L1, L2, L3, L4, L5, TH1: footprint (none) -> Capacitor_SMD:C_0402_1005Metric
- C50: renamed from C58; value 2.2uF -> 4.7uF; footprint (none) -> Capacitor_SMD:C_0402_1005Metric
- C51: renamed from C78; footprint (none) -> Capacitor_SMD:C_0402_1005Metric
- C52: renamed from C65; value 0.1uF -> 100nF; footprint (none) -> Capacitor_SMD:C_0402_1005Metric
- C53: renamed from C59; value 2.2uF -> 4.7uF; footprint (none) -> Capacitor_SMD:C_0402_1005Metric
- C54: renamed from C46; footprint (none) -> Capacitor_SMD:C_0402_1005Metric
- C55: renamed from C68; value 0.1uF -> 100nF; footprint (none) -> Capacitor_SMD:C_0402_1005Metric
- C56: renamed from C66; footprint (none) -> Capacitor_SMD:C_0402_1005Metric
- C57: renamed from C47; value 0.1uF -> 100nF; footprint (none) -> Capacitor_SMD:C_0402_1005Metric
- C58: renamed from C67; value 0.1uF -> 100nF; footprint (none) -> Capacitor_SMD:C_0402_1005Metric
- C59: renamed from C72; value 2.2uF -> 4.7uF; footprint (none) -> Capacitor_SMD:C_0402_1005Metric
- C6: renamed from C81; value 6pF -> 12pF; footprint (none) -> Capacitor_SMD:C_0402_1005Metric
- C60: renamed from C79; footprint (none) -> Capacitor_SMD:C_0402_1005Metric
- C61: renamed from C75; footprint (none) -> Capacitor_SMD:C_0402_1005Metric
- C62: renamed from C80; value 0.1uF -> 100nF; footprint (none) -> Capacitor_SMD:C_0402_1005Metric
- C63: renamed from C70; value 2.2uF -> 4.7uF; footprint (none) -> Capacitor_SMD:C_0402_1005Metric
- C64: renamed from C76; footprint (none) -> Capacitor_SMD:C_0402_1005Metric
- C65: renamed from C44; footprint (none) -> Capacitor_SMD:C_0402_1005Metric
- C66: renamed from C69; footprint (none) -> Capacitor_SMD:C_0402_1005Metric
- C67: renamed from C45; footprint (none) -> Capacitor_SMD:C_0402_1005Metric
- C7: renamed from C82; value 6pF -> 12pF; footprint (none) -> Capacitor_SMD:C_0402_1005Metric
- C73: renamed from C71; value 2.2uF -> 4.7uF; footprint (none) -> Capacitor_SMD:C_0402_1005Metric
- C8: renamed from C83; footprint (none) -> Capacitor_SMD:C_0402_1005Metric
- C9: renamed from C84; footprint (none) -> Capacitor_SMD:C_0402_1005Metric
- L6: value 2nH -> 10uH; footprint (none) -> Capacitor_SMD:C_0402_1005Metric
- R2: renamed from R1; value 3.3k -> 4.7k; footprint (none) -> Capacitor_SMD:C_0402_1005Metric
- R3: renamed from R2; value 3.3k -> 4.7k; footprint (none) -> Capacitor_SMD:C_0402_1005Metric
- R4: value 390k -> 4.7k; footprint (none) -> Capacitor_SMD:C_0402_1005Metric
- R5: renamed from R3; value 390k -> 4.7k; footprint (none) -> Capacitor_SMD:C_0402_1005Metric
- R6: renamed from R5; footprint (none) -> Capacitor_SMD:C_0402_1005Metric
- Y1: value 26MHz -> 32MHz
- renumbered U6 to U2, U7 to U4, U3 to U5, U5 to U7
Connections:
- net CPVIN is gone; now on net AVCC: C66.1, U2.C13 (CPVIN)
- net TP_VCC is gone; now on net IOVCC: U4.11 (TP_VCC), U4.23 (VCI_IN)
- net VCC_DRAM is gone; now on net DCDC4: C22.1, C27.1, C33.1, C36.1, C41.1, C45.1, C61.1, C64.1, R4.1, U2.R10 (VCC_DRAM), U2.R11 (VCC_DRAM), U2.R12 (VCC_DRAM), U2.R13 (VCC_DRAM), U2.R14 (VCC_DRAM), U2.R9 (VCC_DRAM)
- net VCC_EFUSE is gone; now on net AVCC: C38.1, U2.J19 (VCC_EFUSE)
- net VCC_PC is gone; now on net LDO2: C52.1, U2.L18 (VCC_PC)
- net VCC_PD is gone; now on net LDO2: U2.R18 (VCC_PD)
- net VCC_PLL is gone; now on net AVCC: C49.1, U2.N6 (VCC_PLL)
- net VCC_RTC is gone; now on net IOVCC: C44.1, U2.L5 (VCC_RTC)
- net VCC_USB is gone; now on net LDO3: C55.1, U2.J20 (VCC_USB)
- net VCCm is gone; now on net LDO3: C60.1, C62.1, U7.B12 (VCCm), U7.B13 (VCCm), U7.B3 (VCCm), U7.C4 (VCCm), U7.D8 (VCCm)
- net VDD is gone; now on net VDD_SEN: C18.1, C23.1, C29.1, U5.1 (SDO/SA0), U5.2 (SDX), U5.3 (SCX)
- net VDD1 is gone; now on net LDO2: C48.1, C51.1, U7.AA3 (VDD1), U7.AA5 (VDD1), U7.AB3 (VDD1), U7.AB4 (VDD1), U7.AB9 (VDD1), U7.F3 (VDD1), U7.F4 (VDD1), U7.F9 (VDD1), U7.G5 (VDD1)
- net VDD18_DRAM is gone; now on net LDO2: C65.1, C67.1, U2.R15 (VDD18_DRAM)
- net VDD2 is gone; now on net DCDC4: U7.AB5 (VDD2), U7.AB8 (VDD2), U7.F5 (VDD2), U7.F8 (VDD2), U7.J5 (VDD2), U7.K5 (VDD2), U7.L2 (VDD2), U7.L5 (VDD2), U7.M5 (VDD2), U7.N5 (VDD2), U7.P11 (VDD2), U7.P5 (VDD2), U7.P8 (VDD2), U7.R5 (VDD2), U7.T5 (VDD2), U7.U5 (VDD2), U7.V5 (VDD2), U7.W5 (VDD2)
- net VDDCA is gone; now on net DCDC4: U7.K2 (VDDCA), U7.N2 (VDDCA), U7.U2 (VDDCA), U7.V2 (VDDCA)
- net VDDQ is gone; now on net DCDC4: U7.AA9 (VDDQ), U7.G9 (VDDQ), U7.H12 (VDDQ), U7.H8 (VDDQ), U7.J11 (VDDQ), U7.K10 (VDDQ), U7.K12 (VDDQ), U7.L8 (VDDQ), U7.L9 (VDDQ), U7.M10 (VDDQ), U7.M12 (VDDQ), U7.N11 (VDDQ), U7.R11 (VDDQ), U7.T10 (VDDQ), U7.T12 (VDDQ), U7.U8 (VDDQ), U7.U9 (VDDQ), U7.V10 (VDDQ), U7.V12 (VDDQ), U7.W11 (VDDQ), U7.Y12 (VDDQ), U7.Y8 (VDDQ)
- net VDD_CPUS is gone; now on net CPUSLDO: C28.1, U2.N4 (VDD_CPUS)
- net VDD_SYS is gone; now on net DCDC2: C43.1, C46.1, C47.1, C50.1, C53.1, U2.H13 (VDD_SYS), U2.H14 (VDD_SYS), U2.H15 (VDD_SYS), U2.H16 (VDD_SYS), U2.J16 (VDD_SYS)
- net VDD_USB is gone; now on net DCDC2: C17.1, U2.J18 (VDD_USB)
- net 1.8V: now also R2.1, R3.1
- net 32K_IN: now also U3.B9 (P0.00)
- net 32K_OUT: now also U3.B10 (P0.01)
- net AVCC: now also U2.D17 (VCC_MCSI), U2.L4 (VCC_PL), U2.N18 (VCC_LVDS0), C70.1, C71.1, C72.1
- net GND: now also U4.17 (IM0), U5.6 (GND), C19.2, C20.2, C32.2, C35.2, C37.2, C40.2, C42.2, C68.2, C69.2, C70.2, C71.2, C72.2, MIC1.2 (L/R), MIC1.3 (GND), R1.1, U3.B7 (VSS), U3.C1 (VSS_PA), U3.C4 (VSS), U3.D3 (VSS), U3.D4 (VSS), U3.D5 (VSS), U3.D6 (VSS), U3.D7 (VSS), U3.D8 (VSS), U3.E4 (VSS), U3.E5 (VSS), U3.E6 (VSS), U3.E7 (VSS), U3.E8 (VSS), U3.F4 (VSS), U3.F5 (VSS), U3.F6 (VSS), U3.F7 (VSS), U3.F8 (VSS), U3.G4 (VSS), U3.G5 (VSS), U3.G6 (VSS), U3.G7 (VSS), U3.G8 (VSS), U3.K10 (VSS), U6.A1 (VSS)
- net INT_1: now reaches U5.4 (INT1)
- net INT_1: now also U3.C10 (P0.04)
- net SCK: now reaches U4.3 (TP_SCL)
- net SCK: now also R2.2, U1.39 (SCK), U5.13 (SCL), U2.R20 (PD22), U3.K2 (P0.25), U6.A2 (SCL); no longer R3.2
- net SDA: now reaches U4.5 (TP_SDA)
- net SDA: now also R3.2, U1.40 (SDA), U5.14 (SDA), U2.R19 (PD23), U3.K7 (P0.15), U6.B2 (SDA); no longer R2.2
- net CPUSLDO: now reaches U1.10 (CPUSLDO)
- net at L6.2: now also L7.1; no longer C24.1
- net VDD_SEN: now reaches U5.12 (CS)
- net VDD_SEN: now also U5.5 (VDDIO), U5.8 (VDD), U5.9 (INT2), U3.A3 (P1.11), U6.B1 (VDD)
- net 0.9V renamed DCDC2
- net DCDC2: no longer L3.2
- net 1.2V renamed DCDC4
- net 26M_IN renamed 32M_IN
- net 32M_IN: now also U3.A1 (XC1)
- net 26M_OUT renamed 32M_OUT
- net 32M_OUT: now also U3.A2 (XC2)
- removed net 3.3V: L1.2, R2.1, R3.1
- net VCCQm renamed LDO2
- net LDO2: now also C68.1, C69.1
- net VCC_IO renamed LDO3
- net VDDA renamed V_EXT
- net V_EXT: now also C26.1, C19.1, C35.1, U3.B3 (VDD), U3.B8 (VDD), U3.H10 (VDD), U3.K1 (VDD), U3.K5 (VDD)
- net VDDA3P3 renamed DEC4
- net DEC4: now also C24.1, C20.1, U3.A8 (DEC4), U3.C2 (DEC6); no longer C26.1
- net VDD_CPU renamed DCDC3
- net DCDC3: now also L3.2
- new net CS1: U3.K6 (P0.18), U4.6 (CS)
- new net CS2: U2.R22 (SPI1_CS), U3.G1 (P1.07)
- new net DCC: L7.2, U3.A9 (DCC)
- new net DCDC1: L1.2
- new net DEC1: C32.1, U3.A10 (DEC1)
- new net DEC5: C37.1, U3.F2 (DEC5)
- new net DECUSB: U3.K9 (DECUSB)
- new net DSI_CKM: U2.AA23 (DSI_CKM), U4.20 (MIPI_CLKN)
- new net DSI_CKP: U2.AA22 (DSI_CKP), U4.18 (MIPI_CLKP)
- new net DSI_DM0: U2.V23 (DSI_DM0), U4.26 (MIPI_D0N)
- new net DSI_DP0: U2.V22 (DSI_DP0), U4.24 (MIPI_D0P)
- new net D_RST: U3.G10 (P0.12), U4.19 (RESET), U4.21 (PWR_EN), U4.9 (TP_RESET)
- new net IM1: U3.F10 (P1.09), U4.15 (IM1)
- new net INT_2: U3.D10 (P0.05), U4.7 (TP_INT)
- new net MIC_CK: MIC1.4 (CLK)
- new net MIC_D: MIC1.1 (DAT)
- new net MIC_VDD: MIC1.5 (VDD), U3.A4 (P1.13)
- new net NBUS: C42.1, U3.J9 (VBUS)
- new net QSPI_I0: U2.T21 (SPI1_MOSI), U3.J4 (P0.21), U4.14 (SDI0)
- new net QSPI_I1: U2.T22 (SPI_MISO), U3.K3 (P0.22), U4.12 (DCX_SDI1)
- new net QSPI_I2: U3.H5 (P0.23), U4.10 (SDI2)
- new net QSPI_I3: U3.J3 (P1.00), U4.8 (SDI3)
- new net QSPI_SCK: U2.R23 (SPI1_CLK), U3.K4 (P0.19), U4.4 (SCL)
- new net ROT_A: SW1.A, U3.A6 (P0.28)
- new net ROT_B: SW1.B, U3.A5 (P0.03)
- new net SW_0: SW1.S1, U3.A7 (P0.30)
- new net SW_G: R1.2, SW1.C, SW1.S2
- new net nRF_VDD: C40.1, U3.J10 (VDDH)
- no-connect marks 27 -> 35
Other:
- moved on the sheet: C10, C11, C12, C13, C14, C15, C16, C17, C18, C21, C22, C23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
